Commit message: Fix simulation

File: ros/src/sd_gazebo/urdf/r1.gazebo.xacro (robot description, xacro)
@@ -21,4 +21,58 @@
 			<rpyOffsets>0 0 0</rpyOffsets>
 		</plugin>
+	</gazebo>
+	<gazebo>
+		<plugin name="imu_plugin" filename="libgazebo_ros_imu.so">
+			<alwaysOn>true</alwaysOn>
+			<bodyName>base_link</bodyName>
+			<frameName>r1/imu_link</frameName>
+			<topicName>imu/data</topicName>
+			<gaussianNoise>0.0</gaussianNoise>
+			<updateRate>20.0</updateRate>
+			<robotNamespace>/r2</robotNamespace>
+			<serviceName>r1_imu_service</serviceName>
+			<xyzOffset>0 0 0</xyzOffset>
+			<rpyOffset>0 0 0</rpyOffset>
+		</plugin>
+	 </gazebo>
+	<gazebo reference="imu_link">
+		<material>Gazebo/Blue</material>
+	 </gazebo>
+	<gazebo reference="laser_frame">
+		<sensor type="ray" name="head_hokuyo_sensor">
+			<pose>0 0 0 0 0 0</pose>
+			<visualize>false</visualize>
+			<update_rate>40</update_rate>
+			<ray>
+				<scan>
+					<horizontal>
+						<samples>360</samples>
+						<resolution>1</resolution>
+						<min_angle>${-pi}</min_angle>
+						<max_angle>${pi}</max_angle>
+					</horizontal>
+				</scan>
+				<range>
+					<min>0.06</min>
+					<max>5.0</max>
+					<resolution>0.01</resolution>
+				</range>
+				<noise>
+					<type>gaussian</type>
+					<!-- Noise parameters based on published spec for Hokuyo laser
+					achieving "+-30mm" accuracy at range < 10m.  A mean of 0.0m and
+					stddev of 0.01m will put 99.7% of samples within 0.03m of the true
+					reading. -->
+					<mean>0.0</mean>
+					<stddev>0.01</stddev>
+				</noise>
+			</ray>
+			<plugin name="gazebo_ros_head_hokuyo_controller" filename="libgazebo_ros_laser.so">
+				<topicName>laser/scan</topicName>
+				<frameName>laser_frame</frameName>
+				<robotNamespace>/r1</robotNamespace>
+			</plugin>
+		</sensor>
+		<material>Gazebo/Blue</material>
 	</gazebo>
 	<gazebo reference="body_link">

File: ros/src/sd_gazebo/urdf/r2.gazebo.xacro (robot description, xacro)
@@ -31,4 +31,7 @@
 			<updateRate>20.0</updateRate>
 			<robotNamespace>/r2</robotNamespace>
+			<serviceName>r2_imu_service</serviceName>
+			<xyzOffset>0 0 0</xyzOffset>
+			<rpyOffset>0 0 0</rpyOffset>
 		</plugin>
 		<plugin name="mag_plugin" filename="libhector_gazebo_ros_magnetic.so">
