Commit message: Enable controllers

File: ros/src/sd_description/urdf/r2.xacro (robot description, xacro)
@@ -4,5 +4,5 @@
     <xacro:property name="body_width" value="0.260" />
     <xacro:property name="body_height" value="0.424" />
-    <xacro:property name="body_ground_spacing" value="0.01" />
+    <xacro:property name="body_ground_spacing" value="0.005" />
     <xacro:property name="wheel_length" value="0.014" />
     <xacro:property name="wheel_radius" value="0.0375" />

Commit message: Add free wheel

File: ros/src/sd_description/urdf/r2.xacro (robot description, xacro)
@@ -4,5 +4,5 @@
     <xacro:property name="body_width" value="0.260" />
     <xacro:property name="body_height" value="0.424" />
-    <xacro:property name="body_ground_spacing" value="0.005" />
+    <xacro:property name="body_ground_spacing" value="0.010" />
     <xacro:property name="wheel_length" value="0.014" />
     <xacro:property name="wheel_radius" value="0.0375" />
@@ -11,4 +11,5 @@
     <xacro:property name="wheel_velocity_max" value="10000" />
     <xacro:property name="wheel_x" value="0.030" />
+    <xacro:property name="free_wheel_x" value="${-body_length/2 + body_ground_spacing}" />
     <xacro:property name="imu_size" value="0.050"/>
     <xacro:property name="imu_x" value="0.0" />
@@ -83,4 +84,26 @@
     <wheel_macro prefix="left" reflect="1"/>
     <wheel_macro prefix="right" reflect="-1"/>
+    <link name="free_wheel_link">
+        <visual>
+            <geometry>
+                <sphere radius="${body_ground_spacing}"/>
+            </geometry>
+            <material name="black"/>
+        </visual>
+        <collision>
+            <geometry>
+                <sphere radius="${body_ground_spacing}"/>
+            </geometry>
+        </collision>
+        <inertial>
+			<mass value="0.001"/>
+			<inertia ixx="1e-5" ixy="0.0" ixz="0.0" iyy="1e-5" iyz="0.0" izz="1e-5"/>
+        </inertial>
+    </link>
+    <joint name="free_wheel_to_body" type="fixed">
+        <parent link="body_link"/>
+        <child link="free_wheel_link"/>
+        <origin xyz="${free_wheel_x} 0 0" rpy="0 0 0"/>
+    </joint>
     <!-- Sensors -->
     <link name="imu_link">

File: ros/src/sd_gazebo/urdf/r2.gazebo.xacro (robot description, xacro)
@@ -75,4 +75,9 @@
 		<material>Gazebo/Black</material>
 	</gazebo>
+	<gazebo reference="free_wheel_link">
+		<mu1>0.0</mu1>
+		<mu2>0.0</mu2>
+		<material>Gazebo/Black</material>
+	</gazebo>
 	<gazebo>
 		<!--static>true</static-->

Commit message: Add sonar sensor

File: ros/src/sd_description/urdf/r2.xacro (robot description, xacro)
@@ -21,4 +21,9 @@
     <xacro:property name="lidar_y" value="0.0" />
     <xacro:property name="lidar_z" value="0.040" />
+    <xacro:property name="sonar_length" value="0.02"/>
+    <xacro:property name="sonar_width" value="0.044"/>
+    <xacro:property name="sonar_height" value="0.02"/>
+    <xacro:property name="sonar_y" value="0.073"/>
+    <xacro:property name="sonar_z" value="0.120"/>
     <xacro:include filename="$(find sd_description)/urdf/materials.xacro" />
     <link name="base_link"/>
@@ -141,3 +146,20 @@
         <origin xyz="${lidar_x} ${lidar_y} ${lidar_z}" rpy="0 0 0"/>
     </joint>
+    <xacro:macro name="sonar_macro" params="name y">
+        <link name="sonar_${name}_link">
+            <visual>
+                <geometry>
+                    <mesh filename="package://sd_description/meshes/HC-SR04.stl" scale="0.001 0.001 0.001"/>
+                </geometry>
+                <material name="white"/>
+            </visual>
+        </link>
+        <joint name="sonar_${name}_to_body" type="fixed">
+            <parent link="body_link"/>
+            <child link="sonar_${name}_link"/>
+            <origin xyz="${body_length / 2 - sonar_length / 2} ${y} ${sonar_z}" rpy="0 0 0"/>
+        </joint>
+    </xacro:macro>
+    <sonar_macro name="left" y="${sonar_y}"/>
+    <sonar_macro name="right" y="${-sonar_y}"/>
 </robot>

File: ros/src/sd_gazebo/urdf/r2.gazebo.xacro (robot description, xacro)
@@ -72,4 +72,46 @@
 		<material>Gazebo/Blue</material>
 	</gazebo>
+	<xacro:macro name="sonar_sensor_macro" params="name">
+		<gazebo reference="sonar_${name}_link">
+			<sensor type="ray" name="sonar_${name}_sensor">
+				<pose>0 0 0 0 0 0</pose>
+				<update_rate>5</update_rate>
+				<ray>
+					<scan>
+						<horizontal>
+							<samples>5</samples>
+							<resolution>1.0</resolution>
+							<min_angle>-0.0075</min_angle>
+							<max_angle>0.0075</max_angle>
+						</horizontal>
+						<vertical>
+							<samples>5</samples>
+							<resolution>1</resolution>
+							<min_angle>-0.0075</min_angle>
+							<max_angle>0.0075</max_angle>
+						</vertical>
+					</scan>
+					<range>
+						<min>0.08</min>
+						<max>4.0</max>
+						<resolution>0.01</resolution>
+					</range>
+				</ray>
+				<plugin filename="libgazebo_ros_range.so" name="gazebo_ros_range">
+					<gaussianNoise>0.005</gaussianNoise>
+					<alwaysOn>true</alwaysOn>
+					<updateRate>5</updateRate>
+					<topicName>sonar/${name}</topicName>
+					<frameName>r2/sonar_${name}_link</frameName>
+					<fov>0.015</fov>
+					<radiation>ultrasound</radiation>
+					<robotNamespace>/r2</robotNamespace>
+				</plugin>
+			</sensor>
+			<material>Gazebo/White</material>
+		</gazebo>
+	</xacro:macro>
+	<sonar_sensor_macro name="left"/>
+	<sonar_sensor_macro name="right"/>
 	<gazebo reference="body_link">
 		<mu1>0.01</mu1>

Commit message: Lidar is bottom-up

File: ros/src/sd_description/urdf/r2.xacro (robot description, xacro)
@@ -144,5 +144,5 @@
         <parent link="body_link"/>
         <child link="lidar_link"/>
-        <origin xyz="${lidar_x} ${lidar_y} ${lidar_z}" rpy="0 0 0"/>
+        <origin xyz="${lidar_x} ${lidar_y} ${lidar_z}" rpy="${pi} 0 0"/>
     </joint>
     <xacro:macro name="sonar_macro" params="name y">

Commit message: Fix LIDAR orientation

File: ros/src/sd_description/urdf/r2.xacro (robot description, xacro)
@@ -144,5 +144,5 @@
         <parent link="body_link"/>
         <child link="lidar_link"/>
-        <origin xyz="${lidar_x} ${lidar_y} ${lidar_z}" rpy="${pi} 0 0"/>
+        <origin xyz="${lidar_x} ${lidar_y} ${lidar_z}" rpy="${pi} 0 ${pi}"/>
     </joint>
     <xacro:macro name="sonar_macro" params="name y">

Commit message: Update robot description

File: ros/src/sd_description/urdf/r2.xacro (robot description, xacro)
@@ -7,9 +7,9 @@
     <xacro:property name="wheel_length" value="0.014" />
     <xacro:property name="wheel_radius" value="0.0375" />
-    <xacro:property name="wheel_separation" value="0.195" />
+    <xacro:property name="wheel_separation" value="0.190" />
     <xacro:property name="wheel_effort_max" value="10000" />
     <xacro:property name="wheel_velocity_max" value="10000" />
     <xacro:property name="wheel_x" value="0.030" />
-    <xacro:property name="free_wheel_x" value="${-body_length/2 + body_ground_spacing}" />
+    <xacro:property name="free_wheel_x" value="${wheel_x + body_length/2}" />
     <xacro:property name="imu_size" value="0.050"/>
     <xacro:property name="imu_x" value="0.0" />
@@ -18,5 +18,5 @@
     <xacro:property name="lidar_height" value="0.037"/>
     <xacro:property name="lidar_width" value="0.100" />
-    <xacro:property name="lidar_x" value="0.0" />
+    <xacro:property name="lidar_x" value="0.01" />
     <xacro:property name="lidar_y" value="0.0" />
     <xacro:property name="lidar_z" value="0.040" />
@@ -49,5 +49,5 @@
         <parent link="base_link"/>
         <child link="body_link"/>
-        <origin xyz="0 0 ${- wheel_radius + body_ground_spacing}" rpy="0 0 0"/>
+        <origin xyz="${wheel_x} 0 ${- wheel_radius + body_ground_spacing}" rpy="0 0 0"/>
     </joint>
     <xacro:macro name="wheel_macro" params="prefix reflect">
@@ -72,5 +72,5 @@
             <parent link="base_link"/>
             <child link="${prefix}_wheel_link"/>
-            <origin xyz="${wheel_x} ${wheel_separation / 2 * reflect} 0" rpy="${-pi / 2} 0 0"/>
+            <origin xyz="0 ${wheel_separation / 2 * reflect} 0" rpy="${-pi / 2} 0 0"/>
             <limit effort="${wheel_effort_max}" velocity="${wheel_velocity_max}"/>
             <axis xyz="0 0 1"/>
@@ -109,5 +109,5 @@
         <parent link="body_link"/>
         <child link="free_wheel_link"/>
-        <origin xyz="${free_wheel_x} 0 0" rpy="0 0 0"/>
+        <origin xyz="${free_wheel_x} 0 ${body_ground_spacing/2}" rpy="0 0 0"/>
     </joint>
     <!-- Sensors -->

Commit message: Add IMU for R2

File: ros/src/sd_description/urdf/r2.xacro (robot description, xacro)
@@ -13,6 +13,6 @@
     <xacro:property name="free_wheel_x" value="${wheel_x + body_length/2}" />
     <xacro:property name="imu_size" value="0.050"/>
-    <xacro:property name="imu_x" value="0.0" />
-    <xacro:property name="imu_y" value="0.0" />
+    <xacro:property name="imu_x" value="${wheel_x}" />
+    <xacro:property name="imu_y" value="${body_width / 2}" />
     <xacro:property name="imu_z" value="0.170" />
     <xacro:property name="lidar_height" value="0.037"/>
@@ -127,5 +127,5 @@
         <parent link="body_link"/>
         <child link="imu_link"/>
-        <origin xyz="${imu_x} ${imu_y} ${imu_z}" rpy="0 0 0"/>
+        <origin xyz="${imu_x} ${imu_y} ${imu_z}" rpy="0 ${pi} 0"/>
     </joint>
     <link name="lidar_link">

Commit message: Update R2 description (fix LIDAR position)

File: ros/src/sd_description/urdf/r2.xacro (robot description, xacro)
@@ -3,5 +3,5 @@
     <xacro:property name="body_length" value="0.150" />
     <xacro:property name="body_width" value="0.260" />
-    <xacro:property name="body_height" value="0.424" />
+    <xacro:property name="body_height" value="0.350" />
     <xacro:property name="body_ground_spacing" value="0.010" />
     <xacro:property name="wheel_length" value="0.014" />
@@ -10,22 +10,19 @@
     <xacro:property name="wheel_effort_max" value="10000" />
     <xacro:property name="wheel_velocity_max" value="10000" />
-    <xacro:property name="wheel_x" value="0.030" />
-    <xacro:property name="free_wheel_x" value="${wheel_x + body_length/2}" />
+    <xacro:property name="wheel_to_body_x" value="0.030" />
+    <xacro:property name="free_wheel_to_body_x" value="${body_length/2 - 0.012}" />
     <xacro:property name="imu_size" value="0.050"/>
-    <xacro:property name="imu_x" value="${wheel_x}" />
-    <xacro:property name="imu_y" value="${body_width / 2}" />
-    <xacro:property name="imu_z" value="0.170" />
+    <xacro:property name="imu_to_base_x" value="0" />
+    <xacro:property name="imu_to_base_y" value="0" />
+    <xacro:property name="imu_to_base_z" value="${0.145 - wheel_radius}" />
     <xacro:property name="lidar_height" value="0.037"/>
     <xacro:property name="lidar_width" value="0.100" />
-    <xacro:property name="lidar_x" value="0.01" />
-    <xacro:property name="lidar_y" value="0.0" />
-    <xacro:property name="lidar_z" value="0.040" />
-    <xacro:property name="sonar_length" value="0.02"/>
-    <xacro:property name="sonar_width" value="0.044"/>
-    <xacro:property name="sonar_height" value="0.02"/>
-    <xacro:property name="sonar_y" value="0.073"/>
-    <xacro:property name="sonar_z" value="0.120"/>
+    <xacro:property name="lidar_to_base_x" value="-0.04" />
+    <xacro:property name="lidar_to_base_y" value="0.0" />
+    <xacro:property name="lidar_to_base_z" value="${0.040 - wheel_radius}" />
     <xacro:include filename="$(find sd_description)/urdf/materials.xacro" />
+    <!-- Base link is at the center between the wheels axe -->
     <link name="base_link"/>
+    <!-- Body is the robot structure -->
     <link name="body_link">
         <visual>
@@ -49,5 +46,5 @@
         <parent link="base_link"/>
         <child link="body_link"/>
-        <origin xyz="${wheel_x} 0 ${- wheel_radius + body_ground_spacing}" rpy="0 0 0"/>
+        <origin xyz="${wheel_to_body_x} 0 ${- wheel_radius + body_ground_spacing}" rpy="0 0 0"/>
     </joint>
     <xacro:macro name="wheel_macro" params="prefix reflect">
@@ -109,5 +106,5 @@
         <parent link="body_link"/>
         <child link="free_wheel_link"/>
-        <origin xyz="${free_wheel_x} 0 ${body_ground_spacing/2}" rpy="0 0 0"/>
+        <origin xyz="${free_wheel_to_body_x} 0 ${-body_ground_spacing/2}" rpy="0 0 0"/>
     </joint>
     <!-- Sensors -->
@@ -119,13 +116,9 @@
             <material name="blue"/>
         </visual>
-        <!-- <inertial>
-			<mass value="0.1"/>
-			<inertia ixx="0.1e-3" ixy="0.0" ixz="0.0" iyy="0.1e-3" iyz="0.0" izz="0.1e-3"/>
-        </inertial> -->
     </link>
     <joint name="imu_to_body" type="fixed">
-        <parent link="body_link"/>
+        <parent link="base_link"/>
         <child link="imu_link"/>
-        <origin xyz="${imu_x} ${imu_y} ${imu_z}" rpy="0 ${pi} 0"/>
+        <origin xyz="${imu_to_base_x} ${imu_to_base_y} ${imu_to_base_z}" rpy="0 0 0"/>
     </joint>
     <link name="lidar_link">
@@ -136,13 +129,9 @@
             <material name="blue"/>
         </visual>
-        <!-- <inertial>
-			<mass value="0.3"/>
-			<inertia ixx="0.5e-3" ixy="0.0" ixz="0.0" iyy="0.5e-3" iyz="0.0" izz="0.5e-3"/>
-        </inertial> -->
     </link>
     <joint name="lidar_to_body" type="fixed">
-        <parent link="body_link"/>
+        <parent link="base_link"/>
         <child link="lidar_link"/>
-        <origin xyz="${lidar_x} ${lidar_y} ${lidar_z}" rpy="${pi} 0 ${pi}"/>
+        <origin xyz="${lidar_to_base_x} ${lidar_to_base_y} ${lidar_to_base_y}" rpy="0 ${pi} 0"/>
     </joint>
     <xacro:macro name="sonar_macro" params="name y">
@@ -161,5 +150,5 @@
         </joint>
     </xacro:macro>
-    <sonar_macro name="left" y="${sonar_y}"/>
-    <sonar_macro name="right" y="${-sonar_y}"/>
+    <!--sonar_macro name="left" y="${sonar_y}"/-->
+    <!--sonar_macro name="right" y="${-sonar_y}"/-->
 </robot>

Commit message: Fix IMU orientation

File: ros/src/sd_description/urdf/r2.xacro (robot description, xacro)
@@ -120,5 +120,5 @@
         <parent link="base_link"/>
         <child link="imu_link"/>
-        <origin xyz="${imu_to_base_x} ${imu_to_base_y} ${imu_to_base_z}" rpy="0 0 0"/>
+        <origin xyz="${imu_to_base_x} ${imu_to_base_y} ${imu_to_base_z}" rpy="${pi} 0 0"/>
     </joint>
     <link name="lidar_link">
