Commit message: First version of the three wheels drive controller

File: ros/src/sd_description/urdf/r1.xacro (robot description, xacro)
@@ -3,5 +3,5 @@
     <xacro:property name="body_height" value="0.130" />
     <xacro:property name="body_ground_spacing" value="0.01" />
-    <xacro:property name="body_wheels_radius" value="0.162" />
+    <xacro:property name="body_wheel_to_center" value="0.175" />
     <xacro:property name="wheel_length" value="0.034" />
     <xacro:property name="wheel_radius" value="0.030" />
@@ -13,11 +13,12 @@
         <visual>
             <geometry>
-				<mesh filename="package://sd_description/meshes/r1_base.stl" scale="0.001 0.001 0.001"/>
+				<mesh filename="package://sd_description/meshes/r1_base.stl" scale="0.000897 0.000897 0.000897"/>
             </geometry>
             <material name="red"/>
+            <origin xyz="0 0 0" rpy="0 0 ${pi}"/>
         </visual>
         <collision>
             <geometry>
-				<mesh filename="package://sd_description/meshes/r1_base.stl" scale="0.001 0.001 0.001"/>
+				<mesh filename="package://sd_description/meshes/r1_base.stl" scale="0.000897 0.000897 0.000897"/>
             </geometry>
         </collision>
@@ -33,6 +34,6 @@
         <origin xyz="0 0 ${- wheel_radius + body_ground_spacing}" rpy="0 0 0"/>
     </joint>
-    <xacro:macro name="wheel_macro" params="num angle">
-        <link name="wheel_${num}_link">
+    <xacro:macro name="wheel_macro" params="name angle">
+        <link name="${name}_wheel_link">
             <visual>
                 <geometry>
@@ -51,24 +52,24 @@
 	        </inertial>
         </link>
-        <joint name="wheel_${num}_to_base" type="continuous">
+        <joint name="${name}_wheel_to_base" type="continuous">
             <parent link="base_link"/>
-            <child link="wheel_${num}_link"/>
-            <origin xyz="${body_wheels_radius * cos(angle)} ${body_wheels_radius * sin(angle)} 0" rpy="${-pi / 2} 0 ${-pi / 2 + angle}"/>
+            <child link="${name}_wheel_link"/>
+            <origin xyz="${body_wheel_to_center * cos(angle)} ${body_wheel_to_center * sin(angle)} 0" rpy="${-pi / 2} 0 ${pi / 2 + angle}"/>
             <limit effort="${wheel_effort_max}" velocity="${wheel_velocity_max}"/>
             <axis xyz="0 0 1"/>
         </joint>
-		<transmission name="wheel_${num}_to_base_transmission">
+		<transmission name="${name}_wheel_to_base_transmission">
 		    <type>transmission_interface/SimpleTransmission</type>
-		    <joint name="wheel_${num}_to_base">
+		    <joint name="${name}_wheel_to_base">
 				<hardwareInterface>hardware_interface/VelocityJointInterface</hardwareInterface>
 		    </joint>
-		    <actuator name="wheel_${num}_to_base_actuator">
+		    <actuator name="${name}_wheel_to_base_actuator">
 				<hardwareInterface>hardware_interface/VelocityJointInterface</hardwareInterface>
-				<mechanicalReduction>7</mechanicalReduction>
+				<mechanicalReduction>1</mechanicalReduction>
 		    </actuator>
 		</transmission>
     </xacro:macro>
-    <wheel_macro num="1" angle="0"/>
-    <wheel_macro num="2" angle="${2 * pi / 3}"/>
-    <wheel_macro num="3" angle="${-2 * pi / 3}"/>
+    <wheel_macro name="left" angle="${pi / 3}"/>
+    <wheel_macro name="right" angle="${-1 * pi / 3}"/>
+    <wheel_macro name="back" angle="${pi}"/>
 </robot>

File: ros/src/sd_gazebo/urdf/r1.gazebo.xacro (robot description, xacro)
@@ -27,18 +27,18 @@
 		<material>Gazebo/Red</material>
 	</gazebo>
-	<gazebo reference="wheel_1_link">
-		<mu1>100</mu1>
-		<mu2>50</mu2>
+	<gazebo reference="left_wheel_link">
+		<mu1>0.5</mu1>
+		<mu2>0.01</mu2>
 		<material>Gazebo/Black</material>
 	</gazebo>
-	<gazebo reference="wheel_2_link">
-		<mu1>100</mu1>
-		<mu2>50</mu2>
+	<gazebo reference="right_wheel_link">
+		<mu1>0.5</mu1>
+		<mu2>0.01</mu2>
 		<material>Gazebo/Black</material>
 	</gazebo>
-	<gazebo reference="wheel_3_link">
-		<mu1>100</mu1>
-		<mu2>50</mu2>
-		<material>Gazebo/Black</material>
+	<gazebo reference="back_wheel_link">
+		<mu1>0.5</mu1>
+		<mu2>0.01</mu2>
+		<material>Gazebo/Yellow</material>
 	</gazebo>
 	<gazebo>

Commit message: Add realistic simulation for omni wheels

File: ros/src/sd_description/urdf/r1.xacro (robot description, xacro)
@@ -4,6 +4,10 @@
     <xacro:property name="body_ground_spacing" value="0.01" />
     <xacro:property name="body_wheel_to_center" value="0.175" />
-    <xacro:property name="wheel_length" value="0.034" />
-    <xacro:property name="wheel_radius" value="0.030" />
+    <xacro:property name="wheel_length" value="0.026" />
+    <xacro:property name="wheel_radius" value="0.029" />
+    <xacro:property name="wheel_roller_number" value="10" />
+    <xacro:property name="wheel_roller_margin" value="0.001" />
+    <xacro:property name="wheel_roller_radius" value="${wheel_radius/wheel_roller_number}" />
+    <xacro:property name="wheel_roller_length" value="${pi * (wheel_radius - 2 * wheel_roller_radius) / wheel_roller_number}" />
     <xacro:property name="wheel_effort_max" value="10000" />
     <xacro:property name="wheel_velocity_max" value="10000" />
@@ -13,5 +17,5 @@
         <visual>
             <geometry>
-				<mesh filename="package://sd_description/meshes/r1_base.stl" scale="0.000897 0.000897 0.000897"/>
+				<mesh filename="package://sd_description/meshes/r1_base.stl" scale="0.00093 0.00093 0.00093"/>
             </geometry>
             <material name="red"/>
@@ -20,5 +24,5 @@
         <collision>
             <geometry>
-				<mesh filename="package://sd_description/meshes/r1_base.stl" scale="0.000897 0.000897 0.000897"/>
+				<mesh filename="package://sd_description/meshes/r1_base.stl" scale="0.00093 0.00093 0.00093"/>
             </geometry>
         </collision>
@@ -34,9 +38,50 @@
         <origin xyz="0 0 ${- wheel_radius + body_ground_spacing}" rpy="0 0 0"/>
     </joint>
-    <xacro:macro name="wheel_macro" params="name angle">
+    <!-- One roller of the wheel -->
+    <xacro:macro name="roller" params="parent name xyz rpy">
+        <link name="roller_${name}_${parent}_link">
+            <inertial>
+                <mass value="0.002"/>
+                <inertia ixx="2.5e-08" ixy="0" ixz="0" iyy="2.5e-08" iyz="0" izz="1.5e-08"/>
+            </inertial>
+            <visual>
+                <geometry>
+                    <cylinder length="${wheel_roller_length}" radius="${wheel_roller_radius}"/>
+                </geometry>
+                <material name="white"/>
+            </visual>
+            <collision>
+                <geometry>
+                    <cylinder length="${wheel_roller_length}" radius="${wheel_roller_radius}"/>
+                </geometry>
+            </collision>
+        </link>
+        <joint name="roller_${name}_${parent}_to_${parent}" type="continuous">
+            <parent link="${parent}_link"/>
+            <child link="roller_${name}_${parent}_link"/>
+            <axis xyz="0 0 1"/>
+            <origin xyz="${xyz}" rpy="${rpy}" />
+        </joint>
+    </xacro:macro>
+    <!-- Roller loop -->
+    <xacro:macro name="roller_loop" params="parent roller_i z prefix phase">
+        <xacro:if value="${roller_i}">
+            <xacro:roller
+                parent="${parent}" name="${prefix}_${roller_i}"
+                xyz="   ${(wheel_radius - wheel_roller_radius) * cos(phase + 2 * pi * roller_i / wheel_roller_number)}
+                        ${(wheel_radius - wheel_roller_radius) * sin(phase + 2 * pi * roller_i / wheel_roller_number)}
+                        ${z}"
+                rpy="   ${- phase + pi / 2 - 2 * pi * roller_i / wheel_roller_number}
+                        ${pi / 2}
+                        0" />
+            <xacro:roller_loop parent="${parent}" roller_i="${roller_i - 1}" z="${z}" prefix="${prefix}" phase="${phase}"/>
+        </xacro:if>
+    </xacro:macro>
+    <!-- Whell with rollers -->
+    <xacro:macro name="omni_wheel" params="name angle">
         <link name="${name}_wheel_link">
             <visual>
                 <geometry>
-				    <mesh filename="package://sd_description/meshes/r1_wheel.stl" scale="0.001 0.001 0.001"/>
+                    <cylinder length="${wheel_length}" radius="${wheel_radius - 2 * wheel_roller_radius - wheel_roller_margin}"/>
                 </geometry>
                 <material name="black"/>
@@ -44,32 +89,48 @@
             <collision>
                 <geometry>
-                    <cylinder length="${wheel_length}" radius="${wheel_radius}"/>
+                    <cylinder length="${wheel_length}" radius="${wheel_radius - 2 * wheel_roller_radius - wheel_roller_margin}"/>
                 </geometry>
             </collision>
-	        <inertial>
-				<mass value="0.3"/>
-				<inertia ixx="2e-4" ixy="0.0" ixz="0.0" iyy="2e-4" iyz="0.0" izz="2.5e-4"/>
-	        </inertial>
+            <inertial>
+                <mass value="0.3"/>
+                <inertia ixx="2e-4" ixy="0.0" ixz="0.0" iyy="2e-4" iyz="0.0" izz="2.5e-4"/>
+            </inertial>
         </link>
         <joint name="${name}_wheel_to_base" type="continuous">
             <parent link="base_link"/>
             <child link="${name}_wheel_link"/>
-            <origin xyz="${body_wheel_to_center * cos(angle)} ${body_wheel_to_center * sin(angle)} 0" rpy="${-pi / 2} 0 ${pi / 2 + angle}"/>
             <limit effort="${wheel_effort_max}" velocity="${wheel_velocity_max}"/>
             <axis xyz="0 0 1"/>
+            <origin
+                xyz="       ${(body_wheel_to_center - wheel_length / 2) * cos(angle)}
+                            ${(body_wheel_to_center - wheel_length / 2) * sin(angle)}
+                            0"
+                rpy="       ${-pi / 2}
+                            0
+                            ${pi / 2 + angle}"/>
         </joint>
-		<transmission name="${name}_wheel_to_base_transmission">
-		    <type>transmission_interface/SimpleTransmission</type>
-		    <joint name="${name}_wheel_to_base">
-				<hardwareInterface>hardware_interface/VelocityJointInterface</hardwareInterface>
-		    </joint>
-		    <actuator name="${name}_wheel_to_base_actuator">
-				<hardwareInterface>hardware_interface/VelocityJointInterface</hardwareInterface>
-				<mechanicalReduction>1</mechanicalReduction>
-		    </actuator>
-		</transmission>
+        <xacro:roller_loop
+                parent=     "${name}_wheel" prefix="ext"
+                roller_i=   "${wheel_roller_number}"
+                z=          "${wheel_length / 4}"
+                phase=      "${pi / wheel_roller_number}" />
+        <xacro:roller_loop
+                parent=     "${name}_wheel" prefix="int"
+                roller_i=   "${wheel_roller_number}"
+                z=          "${- wheel_length / 4}"
+                phase=       "0" />
+        <transmission name="${name}_wheel_to_base_transmission">
+            <type>transmission_interface/SimpleTransmission</type>
+            <joint name="${name}_wheel_to_base">
+                <hardwareInterface>hardware_interface/VelocityJointInterface</hardwareInterface>
+            </joint>
+            <actuator name="${name}_wheel_to_base_actuator">
+                <hardwareInterface>hardware_interface/VelocityJointInterface</hardwareInterface>
+                <mechanicalReduction>1</mechanicalReduction>
+            </actuator>
+        </transmission>
     </xacro:macro>
-    <wheel_macro name="left" angle="${pi / 3}"/>
-    <wheel_macro name="right" angle="${-1 * pi / 3}"/>
-    <wheel_macro name="back" angle="${pi}"/>
+    <omni_wheel name="left" angle="${pi / 3}"/>
+    <omni_wheel name="right" angle="${-1 * pi / 3}"/>
+    <omni_wheel name="back" angle="${pi}"/>
 </robot>

File: ros/src/sd_gazebo/urdf/r1.gazebo.xacro (robot description, xacro)
@@ -27,21 +27,31 @@
 		<material>Gazebo/Red</material>
 	</gazebo>
-	<gazebo reference="left_wheel_link">
-		<mu1>0.5</mu1>
-		<mu2>0.01</mu2>
-		<material>Gazebo/Black</material>
-	</gazebo>
-	<gazebo reference="right_wheel_link">
-		<mu1>0.5</mu1>
-		<mu2>0.01</mu2>
-		<material>Gazebo/Black</material>
-	</gazebo>
-	<gazebo reference="back_wheel_link">
-		<mu1>0.5</mu1>
-		<mu2>0.01</mu2>
-		<material>Gazebo/Yellow</material>
-	</gazebo>
-	<gazebo>
-		<!--static>true</static-->
-	</gazebo>
+	<!-- One roller of the wheel -->
+    <xacro:macro name="roller_gazebo" params="parent name">
+        <gazebo reference="roller_${name}_${parent}_link">
+	        <mu1>0.5</mu1>
+			<mu2>0.5</mu2>
+			<material>Gazebo/White</material>
+		</gazebo>
+    </xacro:macro>
+    <!-- Roller loop -->
+    <xacro:macro name="roller_loop_gazebo" params="parent roller_i prefix">
+        <xacro:if value="${roller_i}">
+            <xacro:roller_gazebo parent="${parent}" name="${prefix}_${roller_i}" />
+            <xacro:roller_loop_gazebo parent="${parent}" roller_i="${roller_i - 1}" prefix="${prefix}"/>
+        </xacro:if>
+    </xacro:macro>
+    <!-- Whell with rollers -->
+    <xacro:macro name="omni_wheel_gazebo" params="name">
+        <gazebo reference="${name}_wheel_link">
+	        <mu1>0.01</mu1>
+			<mu2>0.01</mu2>
+			<material>Gazebo/Black</material>
+		</gazebo>
+        <xacro:roller_loop_gazebo parent="${name}_wheel" prefix="ext" roller_i="${wheel_roller_number}" />
+        <xacro:roller_loop_gazebo parent="${name}_wheel" prefix="int" roller_i="${wheel_roller_number}" />
+    </xacro:macro>
+    <omni_wheel_gazebo name="left" />
+    <omni_wheel_gazebo name="right" />
+    <omni_wheel_gazebo name="back" />
 </robot>

Commit message: Adapt navigation for r1

File: ros/src/sd_description/urdf/r1.xacro (robot description, xacro)
@@ -63,4 +63,14 @@
             <origin xyz="${xyz}" rpy="${rpy}" />
         </joint>
+        <transmission name="roller_${name}_${parent}_to_${parent}_transmission">
+            <type>transmission_interface/SimpleTransmission</type>
+            <joint name="roller_${name}_${parent}_to_${parent}">
+                <hardwareInterface>hardware_interface/EffortJointInterface</hardwareInterface>
+            </joint>
+            <actuator name="roller_${name}_${parent}_to_${parent}_actuator">
+                <hardwareInterface>hardware_interface/EffortJointInterface</hardwareInterface>
+                <mechanicalReduction>1</mechanicalReduction>
+            </actuator>
+        </transmission>
     </xacro:macro>
     <!-- Roller loop -->

Commit message: Integrate r1 lidar

File: ros/src/sd_description/urdf/r1.xacro (robot description, xacro)
@@ -12,4 +12,8 @@
     <xacro:property name="wheel_effort_max" value="10000" />
     <xacro:property name="wheel_velocity_max" value="10000" />
+    <xacro:property name="lidar_x" value="0.0" />
+    <xacro:property name="lidar_y" value="0.0" />
+    <xacro:property name="lidar_z" value="0.040" />
+    <xacro:property name="lidar_angle" value="${2 * pi / 3}" />
     <xacro:include filename="$(find sd_description)/urdf/materials.xacro" />
     <link name="base_link"/>
@@ -144,3 +148,9 @@
     <omni_wheel name="right" angle="${-1 * pi / 3}"/>
     <omni_wheel name="back" angle="${pi}"/>
+    <xacro:include filename="$(find ydlidar)/urdf/ydlidar.urdf"/>
+    <joint name="lidar_to_body" type="fixed">
+        <parent link="body_link"/>
+        <child link="base_laser"/>
+        <origin xyz="${lidar_x} ${lidar_y} ${lidar_z}" rpy="0 0 ${lidar_angle}"/>
+    </joint>
 </robot>

Commit message: Integrate r1 imu

File: ros/src/sd_description/urdf/r1.xacro (robot description, xacro)
@@ -12,4 +12,7 @@
     <xacro:property name="wheel_effort_max" value="10000" />
     <xacro:property name="wheel_velocity_max" value="10000" />
+    <xacro:property name="imu_x" value="0.0" />
+    <xacro:property name="imu_y" value="0.0" />
+    <xacro:property name="imu_z" value="0.12" />
     <xacro:property name="lidar_x" value="0.0" />
     <xacro:property name="lidar_y" value="0.0" />
@@ -148,4 +151,11 @@
     <omni_wheel name="right" angle="${-1 * pi / 3}"/>
     <omni_wheel name="back" angle="${pi}"/>
+    <link name="imu_link">
+    </link>
+    <joint name="imu_to_body" type="fixed">
+        <parent link="body_link"/>
+        <child link="imu_link"/>
+        <origin xyz="${imu_x} ${imu_y} ${imu_z}" rpy="0 0 0"/>
+    </joint>
     <xacro:include filename="$(find ydlidar)/urdf/ydlidar.urdf"/>
     <joint name="lidar_to_body" type="fixed">

Commit message: Put lidar closer to the ground

File: ros/src/sd_description/urdf/r1.xacro (robot description, xacro)
@@ -17,5 +17,5 @@
     <xacro:property name="lidar_x" value="0.0" />
     <xacro:property name="lidar_y" value="0.0" />
-    <xacro:property name="lidar_z" value="0.040" />
+    <xacro:property name="lidar_z" value="0.020" />
     <xacro:property name="lidar_angle" value="${2 * pi / 3}" />
     <xacro:include filename="$(find sd_description)/urdf/materials.xacro" />

Commit message: Fix IMU origin

File: ros/src/sd_description/urdf/r1.xacro (robot description, xacro)
@@ -156,5 +156,5 @@
         <parent link="body_link"/>
         <child link="imu_link"/>
-        <origin xyz="${imu_x} ${imu_y} ${imu_z}" rpy="0 0 0"/>
+        <origin xyz="${imu_x} ${imu_y} ${imu_z}" rpy="0 ${pi} 0"/>
     </joint>
     <xacro:include filename="$(find ydlidar)/urdf/ydlidar.urdf"/>
